File: raspicam/ir-switcher/ir-switcher.sch (KiCad schematic (older format))
At the start: 11 parts, among them P1 CONN_8, Q1 BC237, Q2 BC237, U1 opto_relay_8, U2 opto_relay_8

Commit message: [raspicam]: Open in new version of KiCad
Parts:
- Q1, Q2: symbol BC237 -> BC237-RESCUE-ir-switcher
- R1, R2, R3, R4: symbol R -> R-RESCUE-ir-switcher
Changed lines of the file:
@@
 EESchema Schematic File Version 2
+LIBS:ir-switcher-rescue
 LIBS:power
 LIBS:device
@@
 LIBS:memory
 LIBS:xilinx
-LIBS:special
 LIBS:microcontrollers
 LIBS:dsp
@@
 LIBS:valves
 LIBS:raspi
-LIBS:raspicam-cache
-EELAYER 24 0
+LIBS:ir-switcher-cache
+EELAYER 25 0
 EELAYER END
 $Descr A4 11693 8268
@@
 $EndDescr
 $Comp
-L R R1
+L R-RESCUE-ir-switcher R1
 U 1 1 5516A622
 P 2850 2600
@@
 $EndComp
 $Comp
-L R R2
+L R-RESCUE-ir-switcher R2
 U 1 1 5516A636
 P 2850 3700
@@
 $EndComp
 $Comp
-L R R4
+L R-RESCUE-ir-switcher R4
 U 1 1 5516A64A
 P 3650 3500
@@
 $EndComp
 $Comp
-L R R3
+L R-RESCUE-ir-switcher R3
 U 1 1 5516A65E
 P 3650 2400
@@
 $EndComp
 $Comp
-L GND #PWR01
+L GND-RESCUE-ir-switcher #PWR01
 U 1 1 5516A9AC
 P 3400 2800
@@
 $EndComp
 $Comp
-L GND #PWR02
+L GND-RESCUE-ir-switcher #PWR02
 U 1 1 5516A9C0
 P 3400 3900
@@
 $EndComp
 $Comp
-L GND #PWR03
+L GND-RESCUE-ir-switcher #PWR03
 U 1 1 5516A9F8
 P 5150 3850
@@
 $EndComp
 $Comp
-L GND #PWR04
+L GND-RESCUE-ir-switcher #PWR04
 U 1 1 55171D54
 P 5150 2050
@@
 $EndComp
 $Comp
-L BC237 Q1
+L BC237-RESCUE-ir-switcher Q1
 U 1 1 5517C071
 P 3300 2600
@@
 $EndComp
 $Comp
-L BC237 Q2
+L BC237-RESCUE-ir-switcher Q2
 U 1 1 5517C1F2
 P 3300 3700
@@
 $EndComp
 $Comp
-L GND #PWR05
+L GND-RESCUE-ir-switcher #PWR05
 U 1 1 5517DF55
 P 1950 3400
@@
 GND
 $Comp
-L GND #PWR06
+L GND-RESCUE-ir-switcher #PWR06
 U 1 1 5517E1BD
 P 2000 1750
@@
 	1650 2250 1900 2250
 $Comp
-L GND #PWR07
+L GND-RESCUE-ir-switcher #PWR07
 U 1 1 5517E2BC
 P 2300 2350
